File: ZVD.kicad_sch (KiCad schematic)
At the start: 4 parts, among them Q1 LMBT5401DW1T1G, Q2 Q_PMOS_GSD

Commit message: minor changes for ERC
Parts:
- Q1: Unit Price 0.04 -> 0.08760924
- Q2: Unit Price 0.04 -> 0.1087452
- R18: Unit Price 0.01 -> 0.0031797
- R19: Unit Price 0.01 -> 0.0137448
Changed lines of the file:
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@@
     (company "Simplexion GmbH")
   )
+  (junction (at 63.5 30.48))
+  (junction (at 48.26 43.18))
+  (junction (at 38.1 50.8))
+  (junction (at 38.1 30.48))
   (junction (at 63.5 50.8))
-  (junction (at 63.5 30.48))
-  (junction (at 38.1 30.48))
-  (junction (at 38.1 50.8))
-  (junction (at 48.26 43.18))
   (wire (pts (xy 35.56 30.48) (xy 38.1 30.48)))
   (wire (pts (xy 38.1 30.48) (xy 45.72 30.48)))
@@
       (effects (font (size 1.27 1.27)) hide)
     )
-    (property "Unit Price" "0.01" (id 5) (at 38.1 57.15 0)
+    (property "Unit Price" "0.0031797" (id 5) (at 38.1 57.15 0)
       (effects (font (size 1.27 1.27)) hide)
     )
@@
       (effects (font (size 1.27 1.27)) hide)
     )
-    (property "Unit Price" "0.01" (id 5) (at 63.5 57.15 0)
+    (property "Unit Price" "0.0137448" (id 5) (at 63.5 57.15 0)
       (effects (font (size 1.27 1.27)) hide)
     )
@@
       (effects (font (size 1.27 1.27)) hide)
     )
-    (property "Unit Price" "0.04" (id 5) (at 40.64 43.18 0)
+    (property "Unit Price" "0.08760924" (id 5) (at 40.64 43.18 0)
       (effects (font (size 1.27 1.27)) hide)
     )
@@
       (effects (font (size 1.27 1.27)) hide)
     )
-    (property "Unit Price" "0.04" (id 5) (at 60.96 43.18 0)
+    (property "Unit Price" "0.08760924" (id 5) (at 60.96 43.18 0)
       (effects (font (size 1.27 1.27)) hide)
     )
@@
       (effects (font (size 1.27 1.27)) hide)
     )
-    (property "Unit Price" "0.04" (id 5) (at 50.8 33.02 0)
+    (property "Unit Price" "0.1087452" (id 5) (at 50.8 33.02 0)
       (effects (font (size 1.27 1.27)) hide)
     )
