File: FT4232HQ.kicad_sch (KiCad schematic)
At the start: 31 parts, among them IC3 USBLC6-2SC6, J4 USB_B_Micro, U15 FT4232H, U3 MCP1703T-3302E/CB, Y2 12MHz

Commit message: cleanup
Parts:
- IC3: value USBLC6-2SC6 -> USBLC6-4SC6
- U15: value FT4232H -> FT4232HQ; MPN (none) -> FT4232HQ-REEL
Other:
- company: Simplexion GmbH -> (none)
- title: FT4232H -> FT4232HQ
Changed lines of the file:
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@@
   (page "A4")
   (title_block
-    (title "FT4232H")
-    (date "2020-04-28")
-    (rev "2.0-rc2")
-    (company "Simplexion GmbH")
-  )
+    (title "FT4232HQ")
+    (date "2020-05-12")
+    (rev "2.0-rc3")
+  )
+  (junction (at 147.32 30.48))
+  (junction (at 184.15 35.56))
+  (junction (at 124.46 63.5))
+  (junction (at 125.73 96.52))
+  (junction (at 114.3 73.66))
+  (junction (at 83.82 35.56))
+  (junction (at 152.4 49.53))
+  (junction (at 24.13 95.25))
+  (junction (at 36.83 78.74))
+  (junction (at 46.99 109.22))
+  (junction (at 167.64 49.53))
+  (junction (at 152.4 161.29))
+  (junction (at 171.45 35.56))
+  (junction (at 45.72 58.42))
+  (junction (at 119.38 35.56))
+  (junction (at 196.85 35.56))
+  (junction (at 116.84 30.48))
+  (junction (at 46.99 83.82))
+  (junction (at 160.02 161.29))
+  (junction (at 114.3 30.48))
+  (junction (at 154.94 49.53))
+  (junction (at 157.48 161.29))
+  (junction (at 142.24 161.29))
+  (junction (at 24.13 106.68))
+  (junction (at 116.84 50.8))
+  (junction (at 154.94 161.29))
+  (junction (at 77.47 109.22))
+  (junction (at 165.1 49.53))
+  (junction (at 149.86 161.29))
+  (junction (at 196.85 45.72))
+  (junction (at 46.99 104.14))
   (junction (at 162.56 161.29))
-  (junction (at 142.24 161.29))
-  (junction (at 45.72 58.42))
-  (junction (at 24.13 95.25))
-  (junction (at 165.1 49.53))
+  (junction (at 184.15 45.72))
+  (junction (at 121.92 35.56))
+  (junction (at 77.47 104.14))
+  (junction (at 119.38 50.8))
+  (junction (at 63.5 58.42))
+  (junction (at 114.3 63.5))
+  (junction (at 124.46 73.66))
+  (junction (at 77.47 86.36))
+  (junction (at 54.61 68.58))
+  (junction (at 83.82 58.42))
   (junction (at 147.32 161.29))
-  (junction (at 184.15 45.72))
-  (junction (at 147.32 30.48))
-  (junction (at 121.92 35.56))
-  (junction (at 116.84 50.8))
-  (junction (at 154.94 49.53))
-  (junction (at 83.82 35.56))
-  (junction (at 184.15 35.56))
-  (junction (at 116.84 30.48))
-  (junction (at 124.46 63.5))
-  (junction (at 124.46 73.66))
-  (junction (at 114.3 63.5))
-  (junction (at 114.3 73.66))
-  (junction (at 54.61 68.58))
-  (junction (at 77.47 104.14))
-  (junction (at 167.64 49.53))
-  (junction (at 119.38 35.56))
-  (junction (at 36.83 78.74))
-  (junction (at 119.38 50.8))
-  (junction (at 46.99 109.22))
-  (junction (at 77.47 109.22))
-  (junction (at 160.02 161.29))
-  (junction (at 154.94 161.29))
-  (junction (at 171.45 35.56))
-  (junction (at 46.99 83.82))
-  (junction (at 77.47 86.36))
-  (junction (at 196.85 45.72))
-  (junction (at 114.3 30.48))
-  (junction (at 149.86 161.29))
-  (junction (at 152.4 49.53))
-  (junction (at 125.73 96.52))
-  (junction (at 157.48 161.29))
-  (junction (at 46.99 104.14))
-  (junction (at 63.5 58.42))
-  (junction (at 24.13 106.68))
-  (junction (at 152.4 161.29))
-  (junction (at 196.85 35.56))
-  (junction (at 83.82 58.42))
+  (no_connect (at 127 124.46))
   (no_connect (at 187.96 152.4))
-  (no_connect (at 187.96 149.86))
-  (no_connect (at 127 124.46))
-  (no_connect (at 34.29 88.9))
   (no_connect (at 127 127))
   (no_connect (at 127 129.54))
+  (no_connect (at 34.29 88.9))
+  (no_connect (at 187.96 149.86))
   (bus_entry (at 198.12 58.42) (size 2.54 -2.54))
   (bus_entry (at 198.12 60.96) (size 2.54 -2.54))
@@
   (bus (pts (xy 200.66 53.34) (xy 200.66 58.42)))
   (bus (pts (xy 200.66 53.34) (xy 203.2 53.34)))
-  (bus (pts (xy 200.66 58.42) (xy 200.66 63.5)))
-  (bus (pts (xy 200.66 63.5) (xy 200.66 68.58)))
-  (bus (pts (xy 200.66 68.58) (xy 200.66 73.66)))
-  (bus (pts (xy 200.66 76.2) (xy 200.66 78.74)))
+  (bus (pts (xy 200.66 58.42) (xy 200.66 60.96)))
+  (bus (pts (xy 200.66 60.96) (xy 200.66 66.04)))
+  (bus (pts (xy 200.66 66.04) (xy 200.66 71.12)))
+  (bus (pts (xy 200.66 71.12) (xy 200.66 73.66)))
+  (bus (pts (xy 200.66 76.2) (xy 200.66 81.28)))
   (bus (pts (xy 200.66 76.2) (xy 203.2 76.2)))
-  (bus (pts (xy 200.66 78.74) (xy 200.66 83.82)))
-  (bus (pts (xy 200.66 83.82) (xy 200.66 88.9)))
-  (bus (pts (xy 200.66 88.9) (xy 200.66 93.98)))
-  (bus (pts (xy 200.66 93.98) (xy 200.66 96.52)))
-  (bus (pts (xy 200.66 99.06) (xy 200.66 104.14)))
+  (bus (pts (xy 200.66 81.28) (xy 200.66 86.36)))
+  (bus (pts (xy 200.66 86.36) (xy 200.66 91.44)))
+  (bus (pts (xy 200.66 91.44) (xy 200.66 96.52)))
+  (bus (pts (xy 200.66 99.06) (xy 200.66 101.6)))
   (bus (pts (xy 200.66 99.06) (xy 203.2 99.06)))
-  (bus (pts (xy 200.66 104.14) (xy 200.66 106.68)))
+  (bus (pts (xy 200.66 101.6) (xy 200.66 106.68)))
   (bus (pts (xy 200.66 106.68) (xy 200.66 111.76)))
   (bus (pts (xy 200.66 111.76) (xy 200.66 116.84)))
   (bus (pts (xy 200.66 116.84) (xy 200.66 119.38)))
-  (bus (pts (xy 200.66 121.92) (xy 200.66 124.46)))
+  (bus (pts (xy 200.66 121.92) (xy 200.66 127)))
   (bus (pts (xy 200.66 121.92) (xy 203.2 121.92)))
-  (bus (pts (xy 200.66 124.46) (xy 200.66 129.54)))
-  (bus (pts (xy 200.66 129.54) (xy 200.66 134.62)))
-  (bus (pts (xy 200.66 134.62) (xy 200.66 139.7)))
-  (bus (pts (xy 200.66 139.7) (xy 200.66 142.24)))
+  (bus (pts (xy 200.66 127) (xy 200.66 132.08)))
+  (bus (pts (xy 200.66 132.08) (xy 200.66 137.16)))
+  (bus (pts (xy 200.66 137.16) (xy 200.66 142.24)))
   (label "D-" (at 44.45 83.82 180)
     (effects (font (size 1.27 1.27)) (justify right bottom))
@@
       (effects (font (size 1.27 1.27)) (justify left))
     )
-    (property "Value" "USBLC6-2SC6" (id 1) (at 68.58 128.27 0)
+    (property "Value" "USBLC6-4SC6" (id 1) (at 68.58 128.27 0)
       (effects (font (size 1.27 1.27)) (justify left))
     )
@@
   (symbol (lib_name "Interface_USB:FT4232H_1") (lib_id "Interface_USB:FT4232H") (at 157.48 106.68 0) (unit 1)
     (property "Reference" "U15" (id 0) (at 157.48 46.3358 0))
-    (property "Value" "FT4232H" (id 1) (at 157.48 48.6345 0))
+    (property "Value" "FT4232HQ" (id 1) (at 157.48 48.6345 0))
     (property "Footprint" "Package_DFN_QFN:QFN-64-1EP_9x9mm_P0.5mm_EP4.7x4.7mm" (id 2) (at 157.48 106.68 0)
       (effects (font (size 1.27 1.27)) hide)
     )
-    (property "Datasheet" "" (id 3) (at 157.48 106.68 0)
+    (property "Datasheet" "https://www.ftdichip.com/Support/Documents/DataSheets/ICs/DS_FT4232H.pdf" (id 3) (at 157.48 106.68 0)
       (effects (font (size 1.27 1.27)) hide)
     )
@@
       (effects (font (size 1.27 1.27)) hide)
     )
+    (property "MPN" "FT4232HQ-REEL" (id 5) (at 157.48 106.68 0)
+      (effects (font (size 1.27 1.27)) hide)
+    )
