File: Blue_Pill.kicad_sch (KiCad schematic)
At the start: 21 parts, among them J14 SWD, SW2 reset, SW3 boot0, U3 STM32F103C8Tx, Y2 8MHz

Commit message: fix USB
Connections:
- net D_N: now also U3.32 (PA11); no longer U3.33 (PA12)
- net D_P: now also U3.33 (PA12); no longer U3.32 (PA11)
Other:
- moved on the sheet: R6, R7
Changed lines of the file:
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@@
 (kicad_sch (version 20200714) (host eeschema "(5.99.0-2360-g1790c536e)")
-  (page 1 5)
+  (page 4 5)
   (paper "A4")
   (title_block
@@
   (junction (at 172.72 43.18) (diameter 0) (color 0 0 0 0))
   (junction (at 172.72 53.34) (diameter 0) (color 0 0 0 0))
-  (junction (at 172.72 106.68) (diameter 0) (color 0 0 0 0))
+  (junction (at 172.72 109.22) (diameter 0) (color 0 0 0 0))
   (junction (at 182.88 43.18) (diameter 0) (color 0 0 0 0))
   (junction (at 182.88 53.34) (diameter 0) (color 0 0 0 0))
+  (no_connect (at 139.7 45.72))
   (no_connect (at 127 73.66))
+  (no_connect (at 160.02 116.84))
   (no_connect (at 127 71.12))
-  (no_connect (at 160.02 116.84))
-  (no_connect (at 139.7 45.72))
   (wire (pts (xy 30.48 40.64) (xy 30.48 41.91))
     (stroke (width 0) (type solid) (color 0 0 0 0))
@@
     (stroke (width 0) (type solid) (color 0 0 0 0))
   )
-  (wire (pts (xy 160.02 106.68) (xy 172.72 106.68))
-    (stroke (width 0) (type solid) (color 0 0 0 0))
-  )
-  (wire (pts (xy 160.02 109.22) (xy 181.61 109.22))
+  (wire (pts (xy 160.02 106.68) (xy 181.61 106.68))
+    (stroke (width 0) (type solid) (color 0 0 0 0))
+  )
+  (wire (pts (xy 160.02 109.22) (xy 172.72 109.22))
     (stroke (width 0) (type solid) (color 0 0 0 0))
   )
@@
     (stroke (width 0) (type solid) (color 0 0 0 0))
   )
-  (wire (pts (xy 172.72 105.41) (xy 172.72 106.68))
-    (stroke (width 0) (type solid) (color 0 0 0 0))
-  )
-  (wire (pts (xy 172.72 106.68) (xy 181.61 106.68))
+  (wire (pts (xy 172.72 105.41) (xy 172.72 109.22))
+    (stroke (width 0) (type solid) (color 0 0 0 0))
+  )
+  (wire (pts (xy 172.72 109.22) (xy 181.61 109.22))
     (stroke (width 0) (type solid) (color 0 0 0 0))
   )
@@
     (effects (font (size 1.27 1.27)) (justify left bottom))
   )
-  (label "D_P" (at 180.34 106.68 180)
+  (label "D_N" (at 180.34 106.68 180)
     (effects (font (size 1.27 1.27)) (justify right bottom))
   )
-  (label "D_N" (at 180.34 109.22 180)
+  (label "D_P" (at 180.34 109.22 180)
     (effects (font (size 1.27 1.27)) (justify right bottom))
   )
@@
     (effects (font (size 1.27 1.27)) (justify left))
   )
-  (hierarchical_label "D+" (shape bidirectional) (at 190.5 106.68 0)
-    (effects (font (size 1.27 1.27)) (justify left))
-  )
-  (hierarchical_label "D-" (shape bidirectional) (at 190.5 109.22 0)
+  (hierarchical_label "D-" (shape bidirectional) (at 190.5 106.68 0)
+    (effects (font (size 1.27 1.27)) (justify left))
+  )
+  (hierarchical_label "D+" (shape bidirectional) (at 190.5 109.22 0)
     (effects (font (size 1.27 1.27)) (justify left))
   )
@@
     )
   )
-  (symbol (lib_id "Device:R") (at 185.42 106.68 90) (mirror x) (unit 1)
-    (in_bom yes) (on_board yes)
-    (property "Reference" "R6" (id 0) (at 185.42 101.4538 90))
-    (property "Value" "20" (id 1) (at 185.42 103.7525 90))
-    (property "Footprint" "Resistor_SMD:R_0603_1608Metric_Icon" (id 2) (at 185.42 104.902 90)
+  (symbol (lib_id "Device:R") (at 185.42 106.68 270) (mirror x) (unit 1)
+    (in_bom yes) (on_board yes)
+    (property "Reference" "R7" (id 0) (at 185.42 102.87 90))
+    (property "Value" "20" (id 1) (at 185.42 100.33 90))
+    (property "Footprint" "Resistor_SMD:R_0603_1608Metric_Icon" (id 2) (at 185.42 108.458 90)
       (effects (font (size 1.27 1.27)) hide)
     )
@@
     )
   )
-  (symbol (lib_id "Device:R") (at 185.42 109.22 270) (unit 1)
-    (in_bom yes) (on_board yes)
-    (property "Reference" "R7" (id 0) (at 185.42 113.03 90))
-    (property "Value" "20" (id 1) (at 185.42 115.57 90))
-    (property "Footprint" "Resistor_SMD:R_0603_1608Metric_Icon" (id 2) (at 185.42 107.442 90)
-      (effects (font (size 1.27 1.27)) hide)
-    )
+  (symbol (lib_id "Device:R") (at 185.42 109.22 90) (unit 1)
+    (in_bom yes) (on_board yes)
+    (property "Reference" "R6" (id 0) (at 185.42 114.4462 90))
+    (property "Value" "20" (id 1) (at 185.42 112.1475 90))
+    (property "Footprint" "Resistor_SMD:R_0603_1608Metric_Icon" (id 2) (at 185.42 110.998 90)
+      (effects (font (size 1.27 1.27)) hide)
+    )
